File: Hardware/KiCad_files/PCIe_interface.sch (KiCad schematic (older format))
At the start: 13 parts, among them J1 PCIe_x4_Connector, U1 XC7A25T_CSG325

Commit message: Upgraded FPGA
Changed FPGA part from XC7A25T to XC7A35T
Parts:
- removed U1: XC7A25T_CSG325, symbol XC7A25T_CSG325
- added U?: XC7A35T_CSG325, symbol XC7A35T_CSG325
Connections:
- net PCIe_CLK_N: now also U?.D5 (MGTREFCLK0N_216)
- net PCIe_CLK_P: now also U?.D6 (MGTREFCLK0P_216)
- net PCIe_RX0_N: now also U?.E3 (MGTPRXN0_216)
- net PCIe_RX0_P: now also U?.E4 (MGTPRXP0_216)
- net PCIe_RX1_N: now also U?.A3 (MGTPRXN1_216)
- net PCIe_RX1_P: now also U?.A4 (MGTPRXP1_216)
- net PCIe_RX2_N: now also U?.C3 (MGTPRXN2_216)
- net PCIe_RX2_P: now also U?.C4 (MGTPRXP2_216)
- net PCIe_RX3_N: now also U?.G3 (MGTPRXN3_216)
- net PCIe_RX3_P: now also U?.G4 (MGTPRXP3_216)
- net PCIe_TX0_N: now also U?.H1 (MGTPTXN0_216)
- net PCIe_TX0_P: now also U?.H2 (MGTPTXP0_216)
- net PCIe_TX1_N: now also U?.F1 (MGTPTXN1_216)
- net PCIe_TX1_P: now also U?.F2 (MGTPTXP1_216)
- net PCIe_TX2_N: now also U?.D1 (MGTPTXN2_216)
- net PCIe_TX2_P: now also U?.D2 (MGTPTXP2_216)
- net PCIe_TX3_N: now also U?.B1 (MGTPTXN3_216)
- net PCIe_TX3_P: now also U?.B2 (MGTPTXP3_216)
- net at R1.1: now also U?.A6 (MGTRREF_216)
Changed lines of the file:
@@
 LIBS:valves
 LIBS:custom
-LIBS:pcie_test_1-cache
+LIBS:RASAC-cache
 EELAYER 25 0
 EELAYER END
@@
 	8600 4500 8500 4500
 $Comp
-L XC7A25T_CSG325 U1
-U 5 1 5C0631C8
+L XC7A35T_CSG325 U?
+U 5 1 5C173C24
 P 7900 4500
-F 0 "U1" H 7900 4200 60  0000 C CNN
-F 1 "XC7A25T_CSG325" H 7900 4300 60  0000 C CNN
+F 0 "U?" H 7900 4200 60  0000 C CNN
+F 1 "XC7A35T_CSG325" H 7900 4300 60  0000 C CNN
 F 2 "" H 8200 6250 60  0001 C CNN
 F 3 "" H 8200 6250 60  0001 C CNN
