File: Hardware/KiCad_files/Power.sch (KiCad schematic (older format))
At the start: 76 parts, among them J2 PCIe_6_Pin_Power, Q1 Q_NMOS_DGS, Q2 Q_PMOS_DGS, U1 XC7A25T_CSG325, U2 PI3420, U3 PI3421, U4 PI3420

Commit message: Upgraded FPGA
Changed FPGA part from XC7A25T to XC7A35T
Parts:
- removed U1: XC7A25T_CSG325, symbol XC7A25T_CSG325
- added U? (x7): XC7A35T_CSG325, symbol XC7A35T_CSG325
Connections:
- net GND: now also U?.A1 (GND), U?.A11 (GND), U?.A18 (GND), U?.A5 (GND), U?.A7 (GND), U?.A8 (GND), U?.B18 (GND), U?.B3 (GND), U?.B7 (GND), U?.B8 (GND), U?.C15 (GND), U?.C2 (GND), U?.C6 (GND), U?.C7 (GND), U?.D12 (GND), U?.D3 (GND), U?.D4 (GND), U?.D7 (GND), U?.E2 (GND), U?.E6 (GND), U?.E7 (GND), U?.E9 (GND), U?.F10 (GND), U?.F16 (GND), U?.F4 (GND), U?.F6 (GND), U?.G1 (GND), U?.G11 (GND), U?.G13 (GND), U?.G5 (GND), U?.G6 (GND), U?.G7 (GND), U?.G9 (GND), U?.H10 (GND), U?.H12 (GND), U?.H3 (GND), U?.H4 (GND), U?.H5 (GND), U?.H6 (GND), U?.H8 (GND), U?.J1 (GND), U?.J11 (GND), U?.J13 (GND), U?.J17 (GND), U?.J2 (GND), U?.J3 (GND), U?.J7 (GND), U?.K12 (GND), U?.K14 (GND), U?.K4 (GND), U?.K8 (GND), U?.L1 (GND), U?.L11 (GND), U?.L13 (GND), U?.L7 (GND), U?.M12 (GND), U?.M18 (GND), U?.M8 (GND), U?.N11 (GND), U?.N13 (GND), U?.N15 (GND), U?.N5 (GND), U?.N7 (GND), U?.N9 (GND), U?.P12 (GND), U?.P2 (GND), U?.P8 (GND), U?.R9 (GND), U?.T16 (GND), U?.T6 (GND), U?.U13 (GND), U?.U3 (GND), U?.V1 (GND), U?.V10 (GND), U?.V18 (GND)
- net MGTAVCC: now also U?.B4 (MGTAVCC), U?.C5 (MGTAVCC), U?.E5 (MGTAVCC), U?.F11 (VCCBRAM), U?.F5 (MGTAVCC), U?.F7 (VCCINT), U?.F9 (VCCINT), U?.G10 (VCCBRAM), U?.G8 (VCCINT), U?.H11 (VCCBRAM), U?.H7 (VCCINT), U?.H9 (VCCINT), U?.J12 (VCCINT), U?.J8 (VCCINT), U?.K11 (VCCINT), U?.K7 (VCCINT), U?.L12 (VCCINT), U?.L8 (VCCINT), U?.M11 (VCCINT), U?.M7 (VCCINT), U?.N10 (VCCINT), U?.N12 (VCCINT), U?.N8 (VCCINT), U?.P11 (VCCINT), U?.P9 (VCCINT)
- net MGTAVTT: now also U?.A2 (MGTAVTT), U?.C1 (MGTAVTT), U?.E1 (MGTAVTT), U?.F3 (MGTAVTT), U?.G2 (MGTAVTT)
- net VCC1V8: now also U?.G12 (VCCAUX), U?.H13 (VCCAUX), U?.K13 (VCCAUX), U?.M13 (VCCAUX), U?.P13 (VCCAUX)
Changed lines of the file:
@@
 LIBS:valves
 LIBS:custom
-LIBS:pcie_test_1-cache
+LIBS:RASAC-cache
 EELAYER 25 0
 EELAYER END
@@
 Text Notes 4000 4850 0    60   ~ 0
 Other power regulators go here
-$Comp
-L XC7A25T_CSG325 U1
-U 12 1 5C0619D0
-P 1150 4800
-F 0 "U1" H 1150 4500 60  0000 C CNN
-F 1 "XC7A25T_CSG325" H 1150 4600 60  0000 C CNN
-F 2 "" H 1450 6550 60  0001 C CNN
-F 3 "" H 1450 6550 60  0001 C CNN
-	12   1150 4800
-	1    0    0    -1
-$EndComp
-$Comp
-L XC7A25T_CSG325 U1
-U 11 1 5C061C0A
-P 1150 3900
-F 0 "U1" H 1150 3600 60  0000 C CNN
-F 1 "XC7A25T_CSG325" H 1150 3700 60  0000 C CNN
-F 2 "" H 1450 5650 60  0001 C CNN
-F 3 "" H 1450 5650 60  0001 C CNN
-	11   1150 3900
-	1    0    0    -1
-$EndComp
-$Comp
-L XC7A25T_CSG325 U1
-U 10 1 5C061DD5
-P 1200 3100
-F 0 "U1" H 1200 2800 60  0000 C CNN
-F 1 "XC7A25T_CSG325" H 1200 2900 60  0000 C CNN
-F 2 "" H 1500 4850 60  0001 C CNN
-F 3 "" H 1500 4850 60  0001 C CNN
-	10   1200 3100
-	1    0    0    -1
-$EndComp
-$Comp
-L XC7A25T_CSG325 U1
-U 9 1 5C0620F5
-P 2600 7200
-F 0 "U1" H 2600 6900 60  0000 C CNN
-F 1 "XC7A25T_CSG325" H 2600 7000 60  0000 C CNN
-F 2 "" H 2900 8950 60  0001 C CNN
-F 3 "" H 2900 8950 60  0001 C CNN
-	9    2600 7200
-	1    0    0    -1
-$EndComp
-$Comp
-L XC7A25T_CSG325 U1
-U 8 1 5C0621BC
-P 1400 7200
-F 0 "U1" H 1400 6900 60  0000 C CNN
-F 1 "XC7A25T_CSG325" H 1400 7000 60  0000 C CNN
-F 2 "" H 1700 8950 60  0001 C CNN
-F 3 "" H 1700 8950 60  0001 C CNN
-	8    1400 7200
-	1    0    0    -1
-$EndComp
-$Comp
-L XC7A25T_CSG325 U1
-U 7 1 5C06228F
-P 2550 4800
-F 0 "U1" H 2550 4500 60  0000 C CNN
-F 1 "XC7A25T_CSG325" H 2550 4600 60  0000 C CNN
-F 2 "" H 2850 6550 60  0001 C CNN
-F 3 "" H 2850 6550 60  0001 C CNN
-	7    2550 4800
-	1    0    0    -1
-$EndComp
-$Comp
-L XC7A25T_CSG325 U1
-U 6 1 5C062364
-P 1150 2400
-F 0 "U1" H 1150 2100 60  0000 C CNN
-F 1 "XC7A25T_CSG325" H 1150 2200 60  0000 C CNN
-F 2 "" H 1450 4150 60  0001 C CNN
-F 3 "" H 1450 4150 60  0001 C CNN
-	6    1150 2400
-	1    0    0    -1
-$EndComp
 Text Notes 8850 3850 0    60   ~ 0
 1.2V Output Following 1.0V
@@
 Text Notes 4500 4250 0    60   ~ 0
 RAM needs 2.5V
+$Comp
+L XC7A35T_CSG325 U?
+U 8 1 5C174146
+P 1400 7200
+F 0 "U?" H 1400 6900 60  0000 C CNN
+F 1 "XC7A35T_CSG325" H 1400 7000 60  0000 C CNN
+F 2 "" H 1700 8950 60  0001 C CNN
+F 3 "" H 1700 8950 60  0001 C CNN
+	8    1400 7200
+	1    0    0    -1
+$EndComp
+$Comp
+L XC7A35T_CSG325 U?
+U 9 1 5C174229
+P 2600 7200
+F 0 "U?" H 2600 6900 60  0000 C CNN
+F 1 "XC7A35T_CSG325" H 2600 7000 60  0000 C CNN
+F 2 "" H 2900 8950 60  0001 C CNN
+F 3 "" H 2900 8950 60  0001 C CNN
+	9    2600 7200
+	1    0    0    -1
+$EndComp
+$Comp
+L XC7A35T_CSG325 U?
+U 10 1 5C1742F8
+P 1200 3100
+F 0 "U?" H 1200 2800 60  0000 C CNN
+F 1 "XC7A35T_CSG325" H 1200 2900 60  0000 C CNN
+F 2 "" H 1500 4850 60  0001 C CNN
+F 3 "" H 1500 4850 60  0001 C CNN
+	10   1200 3100
+	1    0    0    -1
+$EndComp
+$Comp
+L XC7A35T_CSG325 U?
+U 11 1 5C1743D9
+P 1150 3900
+F 0 "U?" H 1150 3600 60  0000 C CNN
+F 1 "XC7A35T_CSG325" H 1150 3700 60  0000 C CNN
+F 2 "" H 1450 5650 60  0001 C CNN
+F 3 "" H 1450 5650 60  0001 C CNN
+	11   1150 3900
+	1    0    0    -1
+$EndComp
+$Comp
+L XC7A35T_CSG325 U?
+U 12 1 5C1744A4
+P 1150 4800
+F 0 "U?" H 1150 4500 60  0000 C CNN
+F 1 "XC7A35T_CSG325" H 1150 4600 60  0000 C CNN
+F 2 "" H 1450 6550 60  0001 C CNN
+F 3 "" H 1450 6550 60  0001 C CNN
+	12   1150 4800
+	1    0    0    -1
+$EndComp
+$Comp
+L XC7A35T_CSG325 U?
+U 6 1 5C1747A8
+P 1150 2400
+F 0 "U?" H 1150 2100 60  0000 C CNN
+F 1 "XC7A35T_CSG325" H 1150 2200 60  0000 C CNN
+F 2 "" H 1450 4150 60  0001 C CNN
+F 3 "" H 1450 4150 60  0001 C CNN
+	6    1150 2400
+	1    0    0    -1
+$EndComp
+$Comp
+L XC7A35T_CSG325 U?
+U 7 1 5C174893
+P 2550 4800
+F 0 "U?" H 2550 4500 60  0000 C CNN
+F 1 "XC7A35T_CSG325" H 2550 4600 60  0000 C CNN
+F 2 "" H 2850 6550 60  0001 C CNN
+F 3 "" H 2850 6550 60  0001 C CNN
+	7    2550 4800
+	1    0    0    -1
+$EndComp
 $EndSCHEMATC

Commit message: Added  HDMI transmitter chip
Also added resistors and moved HDMI data pins around on FPGA side
Other:
- note added: "RAM needs 2.5V\nSYSCLK needs 2.5V"
- note removed: "RAM needs 2.5V"
Changed lines of the file:
@@
 Wire Wire Line
 	5400 4050 5150 4050
-Text Notes 4500 4250 0    60   ~ 0
-RAM needs 2.5V
+Text Notes 4500 4350 0    60   ~ 0
+RAM needs 2.5V\nSYSCLK needs 2.5V
 $Comp
 L XC7A35T_CSG325 U?
