File: KiCad_files/DDR4_1.sch (KiCad schematic (older format))
At the start: 16 parts

Commit message: Cleanup for demo/presentation
Merged Config and Debug sheets.
Added GPIO for remaining pins.
Annotations.
Parts:
- gave numbers to parts that had none: 16
Changed lines of the file:
@@
 $Descr A4 11693 8268
 encoding utf-8
-Sheet 8 10
+Sheet 7 10
 Title "Reconfigurable Application-Specific Accelerator Card"
 Date "2018-11-27"
@@
 $EndDescr
 $Comp
-L EDY4016A J?
+L EDY4016A J5
 U 1 1 5C13D0F3
 P 5900 3900
-F 0 "J?" H 5900 5750 50  0000 C CNN
+F 0 "J5" H 5900 5750 50  0000 C CNN
 F 1 "EDY4016A" H 5850 3900 50  0000 C CNN
 F 2 "" H 5900 2550 50  0001 C CNN
@@
 VCC2V5
 $Comp
-L R_Small R?
+L R_Small R28
 U 1 1 5C144747
 P 4350 1850
-F 0 "R?" H 4380 1870 50  0000 L CNN
+F 0 "R28" H 4380 1870 50  0000 L CNN
 F 1 "240" H 4380 1810 50  0000 L CNN
 F 2 "" H 4350 1850 50  0001 C CNN
@@
 $EndComp
 $Comp
-L GND #PWR?
+L GND #PWR97
 U 1 1 5C144778
 P 4350 1950
-F 0 "#PWR?" H 4350 1700 50  0001 C CNN
+F 0 "#PWR97" H 4350 1700 50  0001 C CNN
 F 1 "GND" H 4350 1800 50  0001 C CNN
 F 2 "" H 4350 1950 50  0001 C CNN
@@
 $EndComp
 $Comp
-L GND #PWR?
+L GND #PWR98
 U 1 1 5C144808
 P 5900 6150
-F 0 "#PWR?" H 5900 5900 50  0001 C CNN
+F 0 "#PWR98" H 5900 5900 50  0001 C CNN
 F 1 "GND" H 5900 6000 50  0001 C CNN
 F 2 "" H 5900 6150 50  0001 C CNN
@@
 $EndComp
 $Comp
-L R R?
+L R R26
 U 1 1 5C144B03
 P 3300 1500
-F 0 "R?" V 3380 1500 50  0000 C CNN
+F 0 "R26" V 3380 1500 50  0000 C CNN
 F 1 "100" V 3300 1500 50  0000 C CNN
 F 2 "" V 3230 1500 50  0001 C CNN
@@
 $EndComp
 $Comp
-L R R?
+L R R27
 U 1 1 5C144B0A
 P 3300 1800
-F 0 "R?" V 3380 1800 50  0000 C CNN
+F 0 "R27" V 3380 1800 50  0000 C CNN
 F 1 "100" V 3300 1800 50  0000 C CNN
 F 2 "" V 3230 1800 50  0001 C CNN
@@
 $EndComp
 $Comp
-L GND #PWR?
+L GND #PWR94
 U 1 1 5C144B11
 P 3300 1950
-F 0 "#PWR?" H 3300 1700 50  0001 C CNN
+F 0 "#PWR94" H 3300 1700 50  0001 C CNN
 F 1 "GND" H 3300 1800 50  0001 C CNN
 F 2 "" H 3300 1950 50  0001 C CNN
@@
 VCC1V2
 $Comp
-L C_Small C?
+L C_Small C95
 U 1 1 5C145216
 P 3050 1800
-F 0 "C?" H 3060 1870 50  0000 L CNN
+F 0 "C95" H 3060 1870 50  0000 L CNN
 F 1 "0.1uF" H 3060 1720 50  0000 L CNN
 F 2 "" H 3050 1800 50  0001 C CNN
@@
 $EndComp
 $Comp
-L C_Small C?
+L C_Small C94
 U 1 1 5C145289
 P 3050 1500
-F 0 "C?" H 3060 1570 50  0000 L CNN
+F 0 "C94" H 3060 1570 50  0000 L CNN
 F 1 "0.1uF" H 3060 1420 50  0000 L CNN
 F 2 "" H 3050 1500 50  0001 C CNN
@@
 VCC1V2
 $Comp
-L GND #PWR?
+L GND #PWR95
 U 1 1 5C14848E
 P 3400 7150
-F 0 "#PWR?" H 3400 6900 50  0001 C CNN
+F 0 "#PWR95" H 3400 6900 50  0001 C CNN
 F 1 "GND" H 3400 7000 50  0001 C CNN
 F 2 "" H 3400 7150 50  0001 C CNN
@@
 $EndComp
 $Comp
-L C_Small C?
+L C_Small C89
 U 1 1 5C1484C9
 P 2350 6700
-F 0 "C?" H 2360 6770 50  0000 L CNN
+F 0 "C89" H 2360 6770 50  0000 L CNN
 F 1 "4.7uF" H 2360 6620 50  0000 L CNN
 F 2 "" H 2350 6700 50  0001 C CNN
@@
 $EndComp
 $Comp
-L C_Small C?
+L C_Small C91
 U 1 1 5C14882E
 P 2650 6700
-F 0 "C?" H 2660 6770 50  0000 L CNN
+F 0 "C91" H 2660 6770 50  0000 L CNN
 F 1 "4.7uF" H 2660 6620 50  0000 L CNN
 F 2 "" H 2650 6700 50  0001 C CNN
@@
 $EndComp
 $Comp
-L C_Small C?
+L C_Small C93
 U 1 1 5C1488A8
 P 2950 6700
-F 0 "C?" H 2960 6770 50  0000 L CNN
+F 0 "C93" H 2960 6770 50  0000 L CNN
 F 1 "4.7uF" H 2960 6620 50  0000 L CNN
 F 2 "" H 2950 6700 50  0001 C CNN
@@
 $EndComp
 $Comp
-L C_Small C?
+L C_Small C97
 U 1 1 5C1488AE
 P 3250 6700
-F 0 "C?" H 3260 6770 50  0000 L CNN
+F 0 "C97" H 3260 6770 50  0000 L CNN
 F 1 "0.068uF" H 3260 6620 50  0000 L CNN
 F 2 "" H 3250 6700 50  0001 C CNN
@@
 $EndComp
 $Comp
-L C_Small C?
+L C_Small C90
 U 1 1 5C148AAE
 P 2500 6950
-F 0 "C?" H 2510 7020 50  0000 L CNN
+F 0 "C90" H 2510 7020 50  0000 L CNN
 F 1 "4.7uF" H 2510 6870 50  0000 L CNN
 F 2 "" H 2500 6950 50  0001 C CNN
@@
 $EndComp
 $Comp
-L C_Small C?
+L C_Small C92
 U 1 1 5C148AB4
 P 2800 6950
-F 0 "C?" H 2810 7020 50  0000 L CNN
+F 0 "C92" H 2810 7020 50  0000 L CNN
 F 1 "4.7uF" H 2810 6870 50  0000 L CNN
 F 2 "" H 2800 6950 50  0001 C CNN
@@
 $EndComp
 $Comp
-L C_Small C?
+L C_Small C96
 U 1 1 5C148ABA
 P 3100 6950
-F 0 "C?" H 3110 7020 50  0000 L CNN
+F 0 "C96" H 3110 7020 50  0000 L CNN
 F 1 "4.7uF" H 3110 6870 50  0000 L CNN
 F 2 "" H 3100 6950 50  0001 C CNN
@@
 $EndComp
 $Comp
-L C_Small C?
+L C_Small C98
 U 1 1 5C148AC0
 P 3400 6950
-F 0 "C?" H 3410 7020 50  0000 L CNN
+F 0 "C98" H 3410 7020 50  0000 L CNN
 F 1 "0.068uF" H 3410 6870 50  0000 L CNN
 F 2 "" H 3400 6950 50  0001 C CNN
@@
 Connection ~ 3250 7100
 $Comp
-L C_Small C?
+L C_Small C99
 U 1 1 5C149C6F
 P 3800 6850
-F 0 "C?" H 3810 6920 50  0000 L CNN
+F 0 "C99" H 3810 6920 50  0000 L CNN
 F 1 "4.7uF" H 3810 6770 50  0000 L CNN
 F 2 "" H 3800 6850 50  0001 C CNN
@@
 $EndComp
 $Comp
-L GND #PWR?
+L GND #PWR96
 U 1 1 5C149CC6
 P 3800 7050
-F 0 "#PWR?" H 3800 6800 50  0001 C CNN
+F 0 "#PWR96" H 3800 6800 50  0001 C CNN
 F 1 "GND" H 3800 6900 50  0001 C CNN
 F 2 "" H 3800 7050 50  0001 C CNN
@@
 $EndComp
 $Comp
-L C_Small C?
+L C_Small C100
 U 1 1 5C149D49
 P 4050 6850
-F 0 "C?" H 4060 6920 50  0000 L CNN
+F 0 "C100" H 4060 6920 50  0000 L CNN
 F 1 "0.1uF" H 4060 6770 50  0000 L CNN
 F 2 "" H 4050 6850 50  0001 C CNN
