File: KiCad_files/HDMI_VGA.sch (KiCad schematic (older format))
At the start: 62 parts, among them J5 TFP410, J6 DB15_Female_HighDensity_Mount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, J7 HDMI_A_1.4, U11 TPD12S521, U12 PCA9306

Commit message: HDMI_VGA is good. Need 5V for HDMI
TODO: DDR2, connections, power
Other:
- note removed: "Unsure about I2C connections and hotplug"
Changed lines of the file:
@@
 $Descr A4 11693 8268
 encoding utf-8
-Sheet 9 10
+Sheet 9 9
 Title "Reconfigurable Application-Specific Accelerator Card"
 Date "2018-11-27"
@@
 Wire Wire Line
 	9200 1900 9200 1600
-Text Notes 5550 4200 0    60   ~ 0
-Unsure about I2C connections and hotplug
 Connection ~ 8900 5850
 Text GLabel 6300 3500 2    60   Input ~ 0

Commit message: Cleanup for DRC and HDMI. HDMI and DDR2 looks good
DRC returns 5 errors with POWEROUTPUT-POWEROUTPUT set as good.
3 of them come from 3V3 since it's being driven from a MOSFET.
1 of them from VCC5V0 not yet supplied.
1 of them from USB_VBUS not set as output.
TODO:
5V supply for HDMI
Connections:
- net VCC3V3: no longer U12.2 (VREF1)
- net VCC5V5 renamed VCC5V0
- new net VCC1V8: U12.2 (VREF1)
Changed lines of the file:
@@
 U 1 1 5C18C3A5
 P 4550 2950
+AR Path="/5C18C3A5" Ref="J5"  Part="1"
+AR Path="/5C14F3D5/5C18C3A5" Ref="J5"  Part="1"
 F 0 "J5" H 5550 4100 50  0000 C CNN
 F 1 "TFP410" H 4550 2950 50  0000 C CNN
@@
 VCC3V3
 Text GLabel 7050 1900 0    60   Input ~ 0
-VCC5V5
+VCC5V0
 $Comp
 L power:GND #PWR0121
@@
 U 1 1 5C60C1C8
 P 8200 1900
+AR Path="/5C60C1C8" Ref="U11"  Part="1"
+AR Path="/5C14F3D5/5C60C1C8" Ref="U11"  Part="1"
 F 0 "U11" H 8200 2167 50  0000 C CNN
 F 1 "TPD12S521" H 8200 2076 50  0000 C CNN
@@
 	9100 3600 9750 3600
 Text GLabel 7600 1250 1    60   Input ~ 0
-VCC5V5
+VCC5V0
 $Comp
 L power:GND #PWR0118
@@
 I2C_SDA
 Text GLabel 4600 6400 1    60   Input ~ 0
-VCC3V3
+VCC1V8
 Text GLabel 9200 1550 1    60   Input ~ 0
 HDMI5V0

Commit message: More caps and added lots of test points
Parts:
- added C? (x2): 1u, symbol Device:C_Small
Connections:
- net GND: now also C?.2, C?.2
- net HDMI5V0: no longer R93.2, R94.2, R95.2, U12.7 (VREF2)
- net VCC3V3: now also C?.1
- net VCC5V0: now also R93.2, R94.2, R95.2, U12.7 (VREF2), C?.1
Changed lines of the file:
@@
 HDMI5V0
 Text GLabel 4800 6400 1    60   Input ~ 0
-HDMI5V0
+VCC5V0
 $Comp
 L Device:R R93
@@
 Wire Wire Line
 	7300 3600 7150 3600
+$Comp
+L Device:C_Small C?
+U 1 1 5C996DF4
+P 6900 1350
+F 0 "C?" H 6992 1396 50  0000 L CNN
+F 1 "1u" H 6992 1305 50  0000 L CNN
+F 2 "" H 6900 1350 50  0001 C CNN
+F 3 "~" H 6900 1350 50  0001 C CNN
+	1    6900 1350
+	1    0    0    -1
+$EndComp
+Text GLabel 6900 1250 1    60   Input ~ 0
+VCC5V0
+$Comp
+L Device:C_Small C?
+U 1 1 5C996DFC
+P 7250 1350
+F 0 "C?" H 7342 1396 50  0000 L CNN
+F 1 "1u" H 7342 1305 50  0000 L CNN
+F 2 "" H 7250 1350 50  0001 C CNN
+F 3 "~" H 7250 1350 50  0001 C CNN
+	1    7250 1350
+	1    0    0    -1
+$EndComp
+Text GLabel 7250 1250 1    60   Input ~ 0
+VCC3V3
+Wire Wire Line
+	7600 1450 7250 1450
+Wire Wire Line
+	7250 1450 6900 1450
+Connection ~ 7250 1450
 $EndSCHEMATC

Commit message: Annotations and proper connections
Parts:
- gave numbers to parts that had none: 2
Changed lines of the file:
@@
 	7300 3600 7150 3600
 $Comp
-L Device:C_Small C?
+L Device:C_Small C228
 U 1 1 5C996DF4
 P 6900 1350
-F 0 "C?" H 6992 1396 50  0000 L CNN
+F 0 "C228" H 6992 1396 50  0000 L CNN
 F 1 "1u" H 6992 1305 50  0000 L CNN
 F 2 "" H 6900 1350 50  0001 C CNN
@@
 VCC5V0
 $Comp
-L Device:C_Small C?
+L Device:C_Small C229
 U 1 1 5C996DFC
 P 7250 1350
-F 0 "C?" H 7342 1396 50  0000 L CNN
+F 0 "C229" H 7342 1396 50  0000 L CNN
 F 1 "1u" H 7342 1305 50  0000 L CNN
 F 2 "" H 7250 1350 50  0001 C CNN
