File: KiCad_files/Decoupling.sch (KiCad schematic (older format))
At the start: 101 parts

Commit message: Finished capacitor footprints
Total cost: ~$55
Parts:
- C100, C101, C102, C103, C106, C107, C109, C110, C111, C112, C113, C114, C117, C118, C119, C120, C121, C122, C123, C124, C126, C127, C128, C129, C130, C131, C132, C135, C136, C137, C138, C139, C140, C143, C144, C145, C146, C147, C150, C151, C160, C161, C170, C171, C179, C180, C87, C88, C89, C90, C91, C92, C95, C96, C98, C99: footprint (none) -> Capacitors_SMD:C_0402
- C104, C115, C93: footprint (none) -> Capacitors_SMD:C_0805
- C105, C116, C125, C133, C149, C153, C154, C155, C156, C157, C159, C163, C164, C165, C166, C167, C168, C169, C172, C173, C174, C175, C176, C177, C178, C181, C182, C183, C184, C185, C186, C86, C94: footprint (none) -> Capacitors_SMD:C_0603
- C108, C134, C141, C97: footprint (none) -> Capacitors_SMD:C_0201
- C142: footprint (none) -> Capacitors_Tantalum_SMD:CP_Tantalum_Case-D_EIA-7343-31_Wave
- C148, C152, C158, C162: footprint (none) -> Capacitors_SMD:C_1210
