File: KiCad_files/Decoupling.sch (KiCad schematic (older format))
At the start: 101 parts

Commit message: Purged RAM (SCH)
Was taking way too lon of a time which I didn't have
Also using larger resistors and capacitors than 0402 and 0201 (expect a very few)
Parts:
- C100, C101, C102, C103, C106, C107, C109, C110, C111, C112, C113, C114, C117, C118, C119, C120, C121, C122, C123, C124, C126, C127, C128, C129, C130, C131, C132, C135, C136, C137, C138, C139, C140, C150, C151, C160, C161, C170, C171, C179, C180, C87, C88, C89, C90, C91, C92, C95, C96, C98, C99: footprint Capacitors_SMD:C_0402 -> Capacitors_SMD:C_0805
- C108, C134, C141, C97: footprint Capacitors_SMD:C_0201 -> Capacitors_SMD:C_0805
- C143, C144, C145, C146, C147: footprint Capacitors_SMD:C_0402 -> Capacitors_SMD:C_0603
