File: KiCad_files/DDR2_1.sch (KiCad schematic (older format))
At the start: 15 parts, among them J10 AS4C128M16D2A

Commit message: Finished capacitor footprints
Total cost: ~$55
Parts:
- C190, C191, C192, C193, C194, C197: footprint (none) -> Capacitors_SMD:C_0603
- C198, C199, C208, C209: footprint (none) -> Capacitors_SMD:C_0201
Changed lines of the file:
@@
 F 0 "C209" H 4810 1870 50  0000 L CNN
 F 1 "0.1uF" H 4810 1720 50  0000 L CNN
-F 2 "" H 4800 1800 50  0001 C CNN
+F 2 "Capacitors_SMD:C_0201" H 4800 1800 50  0001 C CNN
 F 3 "" H 4800 1800 50  0001 C CNN
 	1    4800 1800
@@
 F 0 "C208" H 4810 1570 50  0000 L CNN
 F 1 "0.1uF" H 4810 1420 50  0000 L CNN
-F 2 "" H 4800 1500 50  0001 C CNN
+F 2 "Capacitors_SMD:C_0201" H 4800 1500 50  0001 C CNN
 F 3 "" H 4800 1500 50  0001 C CNN
 	1    4800 1500
@@
 F 0 "C190" H 2360 6770 50  0000 L CNN
 F 1 "4.7uF" H 2360 6620 50  0000 L CNN
-F 2 "" H 2350 6700 50  0001 C CNN
+F 2 "Capacitors_SMD:C_0603" H 2350 6700 50  0001 C CNN
 F 3 "" H 2350 6700 50  0001 C CNN
 	1    2350 6700
@@
 F 0 "C192" H 2660 6770 50  0000 L CNN
 F 1 "4.7uF" H 2660 6620 50  0000 L CNN
-F 2 "" H 2650 6700 50  0001 C CNN
+F 2 "Capacitors_SMD:C_0603" H 2650 6700 50  0001 C CNN
 F 3 "" H 2650 6700 50  0001 C CNN
 	1    2650 6700
@@
 F 0 "C194" H 2960 6770 50  0000 L CNN
 F 1 "4.7uF" H 2960 6620 50  0000 L CNN
-F 2 "" H 2950 6700 50  0001 C CNN
+F 2 "Capacitors_SMD:C_0603" H 2950 6700 50  0001 C CNN
 F 3 "" H 2950 6700 50  0001 C CNN
 	1    2950 6700
@@
 F 0 "C198" H 3260 6770 50  0000 L CNN
 F 1 "0.068uF" H 3260 6620 50  0000 L CNN
-F 2 "" H 3250 6700 50  0001 C CNN
+F 2 "Capacitors_SMD:C_0201" H 3250 6700 50  0001 C CNN
 F 3 "" H 3250 6700 50  0001 C CNN
 	1    3250 6700
@@
 F 0 "C191" H 2510 7020 50  0000 L CNN
 F 1 "4.7uF" H 2510 6870 50  0000 L CNN
-F 2 "" H 2500 6950 50  0001 C CNN
+F 2 "Capacitors_SMD:C_0603" H 2500 6950 50  0001 C CNN
 F 3 "" H 2500 6950 50  0001 C CNN
 	1    2500 6950
@@
 F 0 "C193" H 2810 7020 50  0000 L CNN
 F 1 "4.7uF" H 2810 6870 50  0000 L CNN
-F 2 "" H 2800 6950 50  0001 C CNN
+F 2 "Capacitors_SMD:C_0603" H 2800 6950 50  0001 C CNN
 F 3 "" H 2800 6950 50  0001 C CNN
 	1    2800 6950
@@
 F 0 "C197" H 3110 7020 50  0000 L CNN
 F 1 "4.7uF" H 3110 6870 50  0000 L CNN
-F 2 "" H 3100 6950 50  0001 C CNN
+F 2 "Capacitors_SMD:C_0603" H 3100 6950 50  0001 C CNN
 F 3 "" H 3100 6950 50  0001 C CNN
 	1    3100 6950
@@
 F 0 "C199" H 3410 7020 50  0000 L CNN
 F 1 "0.068uF" H 3410 6870 50  0000 L CNN
-F 2 "" H 3400 6950 50  0001 C CNN
+F 2 "Capacitors_SMD:C_0201" H 3400 6950 50  0001 C CNN
 F 3 "" H 3400 6950 50  0001 C CNN
 	1    3400 6950

Commit message: Almost done with footprints. See issues below
Inductors left to do.
Others without footprints need custom.
PI3420 is out of stock...
LM2676 symbol should be re-drawn for TO-263-7
Total cost: ~$214
Parts:
- J10: footprint (none) -> Housings_BGA:BGA-90_2x3x15_8.0x13.0mm_Pitch0.8mm
- R26, R27: value 100 -> 4.7k; footprint (none) -> Resistors_SMD:R_0402
- TP24, TP25: footprint (none) -> Measurement_Points:Measurement_Point_Round-SMD-Pad_Small
Changed lines of the file:
@@
 P 5050 1500
 F 0 "R26" V 5130 1500 50  0000 C CNN
-F 1 "100" V 5050 1500 50  0000 C CNN
-F 2 "" V 4980 1500 50  0001 C CNN
+F 1 "4.7k" V 5050 1500 50  0000 C CNN
+F 2 "Resistors_SMD:R_0402" V 4980 1500 50  0001 C CNN
 F 3 "" H 5050 1500 50  0001 C CNN
 	1    5050 1500
@@
 P 5050 1800
 F 0 "R27" V 5130 1800 50  0000 C CNN
-F 1 "100" V 5050 1800 50  0000 C CNN
-F 2 "" V 4980 1800 50  0001 C CNN
+F 1 "4.7k" V 5050 1800 50  0000 C CNN
+F 2 "Resistors_SMD:R_0402" V 4980 1800 50  0001 C CNN
 F 3 "" H 5050 1800 50  0001 C CNN
 	1    5050 1800
@@
 F 0 "J10" H 5900 1764 50  0000 C CNN
 F 1 "AS4C128M16D2A" H 5900 1673 50  0000 C CNN
-F 2 "" H 5900 2550 50  0001 C CNN
+F 2 "Housings_BGA:BGA-90_2x3x15_8.0x13.0mm_Pitch0.8mm" H 5900 2550 50  0001 C CNN
 F 3 "" H 5900 2550 50  0001 C CNN
 	1    5900 3900
@@
 F 0 "TP24" H 3458 6624 50  0000 L CNN
 F 1 "TestPoint" H 3458 6579 50  0001 L CNN
-F 2 "" H 3600 6550 50  0001 C CNN
+F 2 "Measurement_Points:Measurement_Point_Round-SMD-Pad_Small" H 3600 6550 50  0001 C CNN
 F 3 "~" H 3600 6550 50  0001 C CNN
 	1    3400 6550
@@
 F 0 "TP25" H 5258 1424 50  0000 L CNN
 F 1 "TestPoint" H 5258 1379 50  0001 L CNN
-F 2 "" H 5400 1350 50  0001 C CNN
+F 2 "Measurement_Points:Measurement_Point_Round-SMD-Pad_Small" H 5400 1350 50  0001 C CNN
 F 3 "~" H 5400 1350 50  0001 C CNN
 	1    5200 1350
