File: KiCad_files/DDR2_2.sch (KiCad schematic (older format))
At the start: 15 parts, among them J11 AS4C128M16D2A

Commit message: Finished capacitor footprints
Total cost: ~$55
Parts:
- C195, C196, C206, C207: footprint (none) -> Capacitors_SMD:C_0201
- C200, C201, C202, C203, C204, C205: footprint (none) -> Capacitors_SMD:C_0603
Changed lines of the file:
@@
 F 0 "C196" H 4810 1870 50  0000 L CNN
 F 1 "0.1uF" H 4810 1720 50  0000 L CNN
-F 2 "" H 4800 1800 50  0001 C CNN
+F 2 "Capacitors_SMD:C_0201" H 4800 1800 50  0001 C CNN
 F 3 "" H 4800 1800 50  0001 C CNN
 	1    4800 1800
@@
 F 0 "C195" H 4810 1570 50  0000 L CNN
 F 1 "0.1uF" H 4810 1420 50  0000 L CNN
-F 2 "" H 4800 1500 50  0001 C CNN
+F 2 "Capacitors_SMD:C_0201" H 4800 1500 50  0001 C CNN
 F 3 "" H 4800 1500 50  0001 C CNN
 	1    4800 1500
@@
 F 0 "C200" H 2360 6770 50  0000 L CNN
 F 1 "4.7uF" H 2360 6620 50  0000 L CNN
-F 2 "" H 2350 6700 50  0001 C CNN
+F 2 "Capacitors_SMD:C_0603" H 2350 6700 50  0001 C CNN
 F 3 "" H 2350 6700 50  0001 C CNN
 	1    2350 6700
@@
 F 0 "C202" H 2660 6770 50  0000 L CNN
 F 1 "4.7uF" H 2660 6620 50  0000 L CNN
-F 2 "" H 2650 6700 50  0001 C CNN
+F 2 "Capacitors_SMD:C_0603" H 2650 6700 50  0001 C CNN
 F 3 "" H 2650 6700 50  0001 C CNN
 	1    2650 6700
@@
 F 0 "C204" H 2960 6770 50  0000 L CNN
 F 1 "4.7uF" H 2960 6620 50  0000 L CNN
-F 2 "" H 2950 6700 50  0001 C CNN
+F 2 "Capacitors_SMD:C_0603" H 2950 6700 50  0001 C CNN
 F 3 "" H 2950 6700 50  0001 C CNN
 	1    2950 6700
@@
 F 0 "C206" H 3260 6770 50  0000 L CNN
 F 1 "0.068uF" H 3260 6620 50  0000 L CNN
-F 2 "" H 3250 6700 50  0001 C CNN
+F 2 "Capacitors_SMD:C_0201" H 3250 6700 50  0001 C CNN
 F 3 "" H 3250 6700 50  0001 C CNN
 	1    3250 6700
@@
 F 0 "C201" H 2510 7020 50  0000 L CNN
 F 1 "4.7uF" H 2510 6870 50  0000 L CNN
-F 2 "" H 2500 6950 50  0001 C CNN
+F 2 "Capacitors_SMD:C_0603" H 2500 6950 50  0001 C CNN
 F 3 "" H 2500 6950 50  0001 C CNN
 	1    2500 6950
@@
 F 0 "C203" H 2810 7020 50  0000 L CNN
 F 1 "4.7uF" H 2810 6870 50  0000 L CNN
-F 2 "" H 2800 6950 50  0001 C CNN
+F 2 "Capacitors_SMD:C_0603" H 2800 6950 50  0001 C CNN
 F 3 "" H 2800 6950 50  0001 C CNN
 	1    2800 6950
@@
 F 0 "C205" H 3110 7020 50  0000 L CNN
 F 1 "4.7uF" H 3110 6870 50  0000 L CNN
-F 2 "" H 3100 6950 50  0001 C CNN
+F 2 "Capacitors_SMD:C_0603" H 3100 6950 50  0001 C CNN
 F 3 "" H 3100 6950 50  0001 C CNN
 	1    3100 6950
@@
 F 0 "C207" H 3410 7020 50  0000 L CNN
 F 1 "0.068uF" H 3410 6870 50  0000 L CNN
-F 2 "" H 3400 6950 50  0001 C CNN
+F 2 "Capacitors_SMD:C_0201" H 3400 6950 50  0001 C CNN
 F 3 "" H 3400 6950 50  0001 C CNN
 	1    3400 6950

Commit message: Almost done with footprints. See issues below
Inductors left to do.
Others without footprints need custom.
PI3420 is out of stock...
LM2676 symbol should be re-drawn for TO-263-7
Total cost: ~$214
Parts:
- J11: footprint (none) -> Housings_BGA:BGA-90_2x3x15_8.0x13.0mm_Pitch0.8mm
- R29, R30: value 100 -> 4.7k; footprint (none) -> Resistors_SMD:R_0402
- TP26, TP27: footprint (none) -> Measurement_Points:Measurement_Point_Round-SMD-Pad_Small
Changed lines of the file:
@@
 P 5050 1500
 F 0 "R29" V 5130 1500 50  0000 C CNN
-F 1 "100" V 5050 1500 50  0000 C CNN
-F 2 "" V 4980 1500 50  0001 C CNN
+F 1 "4.7k" V 5050 1500 50  0000 C CNN
+F 2 "Resistors_SMD:R_0402" V 4980 1500 50  0001 C CNN
 F 3 "" H 5050 1500 50  0001 C CNN
 	1    5050 1500
@@
 P 5050 1800
 F 0 "R30" V 5130 1800 50  0000 C CNN
-F 1 "100" V 5050 1800 50  0000 C CNN
-F 2 "" V 4980 1800 50  0001 C CNN
+F 1 "4.7k" V 5050 1800 50  0000 C CNN
+F 2 "Resistors_SMD:R_0402" V 4980 1800 50  0001 C CNN
 F 3 "" H 5050 1800 50  0001 C CNN
 	1    5050 1800
@@
 F 0 "J11" H 5900 1764 50  0000 C CNN
 F 1 "AS4C128M16D2A" H 5900 1673 50  0000 C CNN
-F 2 "" H 5900 2550 50  0001 C CNN
+F 2 "Housings_BGA:BGA-90_2x3x15_8.0x13.0mm_Pitch0.8mm" H 5900 2550 50  0001 C CNN
 F 3 "" H 5900 2550 50  0001 C CNN
 	1    5900 3900
@@
 F 0 "TP27" H 5258 1424 50  0000 L CNN
 F 1 "TestPoint" H 5258 1379 50  0001 L CNN
-F 2 "" H 5400 1350 50  0001 C CNN
+F 2 "Measurement_Points:Measurement_Point_Round-SMD-Pad_Small" H 5400 1350 50  0001 C CNN
 F 3 "~" H 5400 1350 50  0001 C CNN
 	1    5200 1350
@@
 F 0 "TP26" H 3458 6624 50  0000 L CNN
 F 1 "TestPoint" H 3458 6579 50  0001 L CNN
-F 2 "" H 3600 6550 50  0001 C CNN
+F 2 "Measurement_Points:Measurement_Point_Round-SMD-Pad_Small" H 3600 6550 50  0001 C CNN
 F 3 "~" H 3600 6550 50  0001 C CNN
 	1    3400 6550
