File: KiCad_files/DDR2_2.sch (KiCad schematic (older format))
At the start: 15 parts, among them J11 AS4C128M16D2A

Commit message: Initial FPGA routing + 3D RAM
Slowly losing insanity while listening to WII music for hours
Parts:
- J11: footprint Housings_BGA:BGA-90_2x3x15_8.0x13.0mm_Pitch0.8mm -> custom:BGA-90_2x3x15_8.0x13.0mm_Pitch0.8mm
Changed lines of the file:
@@
 F 0 "J11" H 5900 1764 50  0000 C CNN
 F 1 "AS4C128M16D2A" H 5900 1673 50  0000 C CNN
-F 2 "Housings_BGA:BGA-90_2x3x15_8.0x13.0mm_Pitch0.8mm" H 5900 2550 50  0001 C CNN
+F 2 "custom:BGA-90_2x3x15_8.0x13.0mm_Pitch0.8mm" H 5900 2550 50  0001 C CNN
 F 3 "" H 5900 2550 50  0001 C CNN
 	1    5900 3900
