File: KiCad_files/PCIe_interface.sch (KiCad schematic (older format))
At the start: 13 parts, among them J1 PCIe_x4_Connector, U1 XC7A35T_CSG325

Commit message: Started mapping footprints
Parts:
- C1, C10, C2, C3, C4, C5, C6, C7, C8, C9: footprint (none) -> Capacitors_SMD:C_0402
Changed lines of the file:
@@
 F 0 "C1" H 5760 3520 50  0000 L CNN
 F 1 "0.01uF" H 5760 3370 50  0000 L BNN
-F 2 "" H 5750 3450 50  0001 C CNN
+F 2 "Capacitors_SMD:C_0402" H 5750 3450 50  0001 C CNN
 F 3 "" H 5750 3450 50  0001 C CNN
 	1    5750 3450
@@
 F 0 "C2" H 5760 3720 50  0000 L CNN
 F 1 "0.01uF" H 5760 3570 50  0000 L TNN
-F 2 "" H 5750 3650 50  0001 C CNN
+F 2 "Capacitors_SMD:C_0402" H 5750 3650 50  0001 C CNN
 F 3 "" H 5750 3650 50  0001 C CNN
 	1    5750 3650
@@
 F 0 "C3" H 6110 3820 50  0000 L CNN
 F 1 "0.22uF" H 6110 3670 50  0000 L BNN
-F 2 "" H 6100 3750 50  0001 C CNN
+F 2 "Capacitors_SMD:C_0402" H 6100 3750 50  0001 C CNN
 F 3 "" H 6100 3750 50  0001 C CNN
 	1    6100 3750
@@
 F 0 "C4" H 6110 4020 50  0000 L CNN
 F 1 "0.22uF" H 6110 3870 50  0000 L TNN
-F 2 "" H 6100 3950 50  0001 C CNN
+F 2 "Capacitors_SMD:C_0402" H 6100 3950 50  0001 C CNN
 F 3 "" H 6100 3950 50  0001 C CNN
 	1    6100 3950
@@
 F 0 "C5" H 6110 4320 50  0000 L CNN
 F 1 "0.22uF" H 6110 4170 50  0000 L BNN
-F 2 "" H 6100 4250 50  0001 C CNN
+F 2 "Capacitors_SMD:C_0402" H 6100 4250 50  0001 C CNN
 F 3 "" H 6100 4250 50  0001 C CNN
 	1    6100 4250
@@
 F 0 "C6" H 6110 4520 50  0000 L CNN
 F 1 "0.22uF" H 6110 4370 50  0000 L TNN
-F 2 "" H 6100 4450 50  0001 C CNN
+F 2 "Capacitors_SMD:C_0402" H 6100 4450 50  0001 C CNN
 F 3 "" H 6100 4450 50  0001 C CNN
 	1    6100 4450
@@
 F 0 "C7" H 6110 4720 50  0000 L CNN
 F 1 "0.22uF" H 6110 4570 50  0000 L BNN
-F 2 "" H 6100 4650 50  0001 C CNN
+F 2 "Capacitors_SMD:C_0402" H 6100 4650 50  0001 C CNN
 F 3 "" H 6100 4650 50  0001 C CNN
 	1    6100 4650
@@
 F 0 "C8" H 6110 4920 50  0000 L CNN
 F 1 "0.22uF" H 6110 4770 50  0000 L TNN
-F 2 "" H 6100 4850 50  0001 C CNN
+F 2 "Capacitors_SMD:C_0402" H 6100 4850 50  0001 C CNN
 F 3 "" H 6100 4850 50  0001 C CNN
 	1    6100 4850
@@
 F 0 "C9" H 6110 5120 50  0000 L CNN
 F 1 "0.22uF" H 6110 4970 50  0000 L BNN
-F 2 "" H 6100 5050 50  0001 C CNN
+F 2 "Capacitors_SMD:C_0402" H 6100 5050 50  0001 C CNN
 F 3 "" H 6100 5050 50  0001 C CNN
 	1    6100 5050
@@
 F 0 "C10" H 6110 5320 50  0000 L CNN
 F 1 "0.22uF" H 6110 5170 50  0000 L TNN
-F 2 "" H 6100 5250 50  0001 C CNN
+F 2 "Capacitors_SMD:C_0402" H 6100 5250 50  0001 C CNN
 F 3 "" H 6100 5250 50  0001 C CNN
 	1    6100 5250

Commit message: Almost done with footprints. See issues below
Inductors left to do.
Others without footprints need custom.
PI3420 is out of stock...
LM2676 symbol should be re-drawn for TO-263-7
Total cost: ~$214
Parts:
- J1: footprint (none) -> custom:PCIe_x4
- R1: footprint (none) -> Resistors_SMD:R_0402
Changed lines of the file:
@@
 F 0 "J1" H 4150 5650 50  0000 C CNN
 F 1 "PCIe_x4_Connector" H 4150 2000 50  0000 C CNN
-F 2 "" H 4150 2450 50  0001 C CNN
+F 2 "custom:PCIe_x4" H 4150 2450 50  0001 C CNN
 F 3 "" H 4150 2450 50  0001 C CNN
 	1    4150 3800
@@
 F 0 "R1" V 8730 2500 50  0000 C CNN
 F 1 "100" V 8650 2500 50  0000 C CNN
-F 2 "" V 8580 2500 50  0001 C CNN
+F 2 "Resistors_SMD:R_0402" V 8580 2500 50  0001 C CNN
 F 3 "" H 8650 2500 50  0001 C CNN
 	1    8650 2500

Commit message: Drew FPGA and HDMI footprints
Ready for layout...?
Parts:
- U1: footprint (none) -> custom:BGA-324_15.0x15.0mm_Layout18x18_P0.8mm_Ball0.5mm_Pad0.4mm_NSMD
Changed lines of the file:
@@
 F 0 "U1" H 7900 4200 60  0000 C CNN
 F 1 "XC7A35T_CSG325" H 7900 4300 60  0000 C CNN
-F 2 "" H 8200 6250 60  0001 C CNN
+F 2 "custom:BGA-324_15.0x15.0mm_Layout18x18_P0.8mm_Ball0.5mm_Pad0.4mm_NSMD" H 8200 6250 60  0001 C CNN
 F 3 "" H 8200 6250 60  0001 C CNN
 	5    7900 4500

Commit message: Replaced PCIe x4 footprint
Footprint generated with https://github.com/dlharmon/footgen
Parts:
- J1: footprint custom:PCIe_x4 -> custom:pciex4fingers
Changed lines of the file:
@@
 F 0 "J1" H 4150 5650 50  0000 C CNN
 F 1 "PCIe_x4_Connector" H 4150 2000 50  0000 C CNN
-F 2 "custom:PCIe_x4" H 4150 2450 50  0001 C CNN
+F 2 "custom:pciex4fingers" H 4150 2450 50  0001 C CNN
 F 3 "" H 4150 2450 50  0001 C CNN
 	1    4150 3800
