File: KiCad_files/Connections.sch (KiCad schematic (older format))
At the start: 7 parts, among them U1 XC7A35T_CSG325

Commit message: Finished capacitor footprints
Total cost: ~$55
Parts:
- C187, C188, C189, C225, C226, C227: footprint (none) -> Capacitors_SMD:C_1210
Changed lines of the file:
@@
 F 0 "C187" H 1325 7300 50  0000 L CNN
 F 1 "100uF" H 1325 7100 50  0000 L CNN
-F 2 "" H 1338 7050 50  0001 C CNN
+F 2 "Capacitors_SMD:C_1210" H 1338 7050 50  0001 C CNN
 F 3 "" H 1300 7200 50  0001 C CNN
 	1    1300 7200
@@
 F 0 "C188" H 1925 7300 50  0000 L CNN
 F 1 "100uF" H 1925 7100 50  0000 L CNN
-F 2 "" H 1938 7050 50  0001 C CNN
+F 2 "Capacitors_SMD:C_1210" H 1938 7050 50  0001 C CNN
 F 3 "" H 1900 7200 50  0001 C CNN
 	1    1900 7200
@@
 F 0 "C189" H 2525 7300 50  0000 L CNN
 F 1 "100uF" H 2525 7100 50  0000 L CNN
-F 2 "" H 2538 7050 50  0001 C CNN
+F 2 "Capacitors_SMD:C_1210" H 2538 7050 50  0001 C CNN
 F 3 "" H 2500 7200 50  0001 C CNN
 	1    2500 7200
@@
 F 0 "C227" H 2825 7300 50  0000 L CNN
 F 1 "100uF" H 2825 7100 50  0000 L CNN
-F 2 "" H 2838 7050 50  0001 C CNN
+F 2 "Capacitors_SMD:C_1210" H 2838 7050 50  0001 C CNN
 F 3 "" H 2800 7200 50  0001 C CNN
 	1    2800 7200
@@
 F 0 "C226" H 2225 7300 50  0000 L CNN
 F 1 "100uF" H 2225 7100 50  0000 L CNN
-F 2 "" H 2238 7050 50  0001 C CNN
+F 2 "Capacitors_SMD:C_1210" H 2238 7050 50  0001 C CNN
 F 3 "" H 2200 7200 50  0001 C CNN
 	1    2200 7200
@@
 F 0 "C225" H 1625 7300 50  0000 L CNN
 F 1 "100uF" H 1625 7100 50  0000 L CNN
-F 2 "" H 1638 7050 50  0001 C CNN
+F 2 "Capacitors_SMD:C_1210" H 1638 7050 50  0001 C CNN
 F 3 "" H 1600 7200 50  0001 C CNN
 	1    1600 7200

Commit message: Drew FPGA and HDMI footprints
Ready for layout...?
Parts:
- U1: footprint (none) -> custom:BGA-324_15.0x15.0mm_Layout18x18_P0.8mm_Ball0.5mm_Pad0.4mm_NSMD
Changed lines of the file:
@@
 F 0 "U1" H 2200 5700 60  0000 C CNN
 F 1 "XC7A35T_CSG325" H 2200 5800 60  0000 C CNN
-F 2 "" H 2500 7750 60  0001 C CNN
+F 2 "custom:BGA-324_15.0x15.0mm_Layout18x18_P0.8mm_Ball0.5mm_Pad0.4mm_NSMD" H 2500 7750 60  0001 C CNN
 F 3 "" H 2500 7750 60  0001 C CNN
 	2    2200 6000
@@
 F 0 "U1" H 5600 5700 60  0000 C CNN
 F 1 "XC7A35T_CSG325" H 5600 5800 60  0000 C CNN
-F 2 "" H 5900 7750 60  0001 C CNN
+F 2 "custom:BGA-324_15.0x15.0mm_Layout18x18_P0.8mm_Ball0.5mm_Pad0.4mm_NSMD" H 5900 7750 60  0001 C CNN
 F 3 "" H 5900 7750 60  0001 C CNN
 	3    5600 6000
@@
 F 0 "U1" H 8700 5700 60  0000 C CNN
 F 1 "XC7A35T_CSG325" H 8700 5800 60  0000 C CNN
-F 2 "" H 9000 7750 60  0001 C CNN
+F 2 "custom:BGA-324_15.0x15.0mm_Layout18x18_P0.8mm_Ball0.5mm_Pad0.4mm_NSMD" H 9000 7750 60  0001 C CNN
 F 3 "" H 9000 7750 60  0001 C CNN
 	4    8700 6000
