File: KiCad_files/Power.sch (KiCad schematic (older format))
At the start: 101 parts, among them J2 PCIe_6_Pin_Power, Q1 Q_NMOS_GSD, Q2 Q_PMOS_GSD, U1 XC7A35T_CSG325, U13 LM2676-KTW, U2 MAX15027, U3 PI3420, U4 PI3421, U5 PI3420

Commit message: Fixes during layout
Changed FT2232HL footprint to one with external pad
Made LGA123 (PI34XX) pins into blocks
Added labels for PCIe to let KiCad do differential pair routing
Removed some ground connections in SGND in PI34XX
Connections:
- net GND: no longer R6.2, U3.BLK1 (SGND), U3.K5 (SYNCI), U4.BLK1 (SGND), U4.K5 (SYNCI), U5.BLK1 (SGND), U5.K5 (SYNCI)
- new net SGND_PI3420_1: U3.BLK1 (SGND), U3.K5 (SYNCI)
- new net SGND_PI3420_2: R6.2, U5.BLK1 (SGND), U5.K5 (SYNCI)
- new net SGND_PI3421_1: U4.BLK1 (SGND), U4.K5 (SYNCI)
Changed lines of the file:
@@
 	9900 1000 10000 1000
-Wire Wire Line
-	10000 1500 9950 1500
 Wire Wire Line
 	6650 1600 6750 1600
@@
 	10000 2700 9900 2700
 Wire Wire Line
-	10000 3100 9950 3100
-Wire Wire Line
 	6650 3200 6750 3200
 Wire Wire Line
@@
 Wire Wire Line
 	10000 4300 9900 4300
-Wire Wire Line
-	10000 4700 9950 4700
 Wire Wire Line
 	6650 4800 6750 4800
@@
 	5800 3450 5650 3450
 Connection ~ 5650 3450
-$Comp
-L power:GND #PWR0122
-U 1 1 5C8C264C
-P 9950 1500
-F 0 "#PWR0122" H 9950 1250 50  0001 C CNN
-F 1 "GND" H 9950 1350 50  0001 C CNN
-F 2 "" H 9950 1500 50  0001 C CNN
-F 3 "" H 9950 1500 50  0001 C CNN
-	1    9950 1500
-	1    0    0    -1
-$EndComp
-Connection ~ 9950 1500
-Wire Wire Line
-	9950 1500 9900 1500
-$Comp
-L power:GND #PWR0123
-U 1 1 5C8C27F3
-P 9950 3100
-F 0 "#PWR0123" H 9950 2850 50  0001 C CNN
-F 1 "GND" H 9950 2950 50  0001 C CNN
-F 2 "" H 9950 3100 50  0001 C CNN
-F 3 "" H 9950 3100 50  0001 C CNN
-	1    9950 3100
-	1    0    0    -1
-$EndComp
-Connection ~ 9950 3100
-Wire Wire Line
-	9950 3100 9900 3100
-$Comp
-L power:GND #PWR0130
-U 1 1 5C8C2AA0
-P 9950 4700
-F 0 "#PWR0130" H 9950 4450 50  0001 C CNN
-F 1 "GND" H 9950 4550 50  0001 C CNN
-F 2 "" H 9950 4700 50  0001 C CNN
-F 3 "" H 9950 4700 50  0001 C CNN
-	1    9950 4700
-	1    0    0    -1
-$EndComp
-Connection ~ 9950 4700
-Wire Wire Line
-	9950 4700 9900 4700
 Wire Wire Line
 	9700 5950 9850 5950
@@
 	1    0    0    -1
 $EndComp
+Wire Wire Line
+	9900 4700 10000 4700
+Wire Wire Line
+	9900 3100 10000 3100
+Wire Wire Line
+	9900 1500 10000 1500
 $EndSCHEMATC

Commit message: Purged RAM (SCH)
Was taking way too lon of a time which I didn't have
Also using larger resistors and capacitors than 0402 and 0201 (expect a very few)
Parts:
- C13, C212, C51, C52, C53, C55, C57, C59: footprint Capacitors_SMD:C_0402 -> Capacitors_SMD:C_0805
- C213: footprint Capacitors_SMD:C_0201 -> Capacitors_SMD:C_1206
- C60, C61, C62: footprint Capacitors_SMD:C_0201 -> Capacitors_SMD:C_0805
- R2, R4, R6: footprint Resistors_SMD:R_0402 -> Resistors_SMD:R_0805
Changed lines of the file:
@@
 $Descr A4 11693 8268
 encoding utf-8
-Sheet 3 9
+Sheet 3 7
 Title "Reconfigurable Application-Specific Accelerator Card"
-Date "2019-02-27"
-Rev "1.0"
+Date "2019-03-31"
+Rev "0.9"
 Comp "Brian Hong & Jasmine Tang"
 Comment1 ""
@@
 F 0 "R2" V 2930 1200 50  0000 C CNN
 F 1 "2.2k" V 2850 1200 50  0000 C CNN
-F 2 "Resistors_SMD:R_0402" V 2780 1200 50  0001 C CNN
+F 2 "Resistors_SMD:R_0805" V 2780 1200 50  0001 C CNN
 F 3 "" H 2850 1200 50  0001 C CNN
 	1    2850 1200
@@
 F 0 "C51" H 7960 1870 50  0000 L CNN
 F 1 "1uF" H 7960 1720 50  0000 L CNN
-F 2 "Capacitors_SMD:C_0402" H 7950 1800 50  0001 C CNN
+F 2 "Capacitors_SMD:C_0805" H 7950 1800 50  0001 C CNN
 F 3 "" H 7950 1800 50  0001 C CNN
 	1    7950 1800
@@
 F 0 "C55" H 8110 1870 50  0000 L CNN
 F 1 "1uF" H 8110 1720 50  0000 L CNN
-F 2 "Capacitors_SMD:C_0402" H 8100 1800 50  0001 C CNN
+F 2 "Capacitors_SMD:C_0805" H 8100 1800 50  0001 C CNN
 F 3 "" H 8100 1800 50  0001 C CNN
 	1    8100 1800
@@
 F 0 "C60" H 8260 1870 50  0000 L CNN
 F 1 "0.1uF" H 8260 1720 50  0000 L CNN
-F 2 "Capacitors_SMD:C_0201" H 8250 1800 50  0001 C CNN
+F 2 "Capacitors_SMD:C_0805" H 8250 1800 50  0001 C CNN
 F 3 "" H 8250 1800 50  0001 C CNN
 	1    8250 1800
@@
 F 0 "C52" H 7960 3470 50  0000 L CNN
 F 1 "1uF" H 7960 3320 50  0000 L CNN
-F 2 "Capacitors_SMD:C_0402" H 7950 3400 50  0001 C CNN
+F 2 "Capacitors_SMD:C_0805" H 7950 3400 50  0001 C CNN
 F 3 "" H 7950 3400 50  0001 C CNN
 	1    7950 3400
@@
 F 0 "C57" H 8110 3470 50  0000 L CNN
 F 1 "1uF" H 8110 3320 50  0000 L CNN
-F 2 "Capacitors_SMD:C_0402" H 8100 3400 50  0001 C CNN
+F 2 "Capacitors_SMD:C_0805" H 8100 3400 50  0001 C CNN
 F 3 "" H 8100 3400 50  0001 C CNN
 	1    8100 3400
@@
 F 0 "C61" H 8260 3470 50  0000 L CNN
 F 1 "0.1uF" H 8260 3320 50  0000 L CNN
-F 2 "Capacitors_SMD:C_0201" H 8250 3400 50  0001 C CNN
+F 2 "Capacitors_SMD:C_0805" H 8250 3400 50  0001 C CNN
 F 3 "" H 8250 3400 50  0001 C CNN
 	1    8250 3400
@@
 F 0 "C53" H 7960 5070 50  0000 L CNN
 F 1 "1uF" H 7960 4920 50  0000 L CNN
-F 2 "Capacitors_SMD:C_0402" H 7950 5000 50  0001 C CNN
+F 2 "Capacitors_SMD:C_0805" H 7950 5000 50  0001 C CNN
 F 3 "" H 7950 5000 50  0001 C CNN
 	1    7950 5000
@@
 F 0 "C59" H 8110 5070 50  0000 L CNN
 F 1 "1uF" H 8110 4920 50  0000 L CNN
-F 2 "Capacitors_SMD:C_0402" H 8100 5000 50  0001 C CNN
+F 2 "Capacitors_SMD:C_0805" H 8100 5000 50  0001 C CNN
 F 3 "" H 8100 5000 50  0001 C CNN
 	1    8100 5000
@@
 F 0 "C62" H 8260 5070 50  0000 L CNN
 F 1 "0.1uF" H 8260 4920 50  0000 L CNN
-F 2 "Capacitors_SMD:C_0201" H 8250 5000 50  0001 C CNN
+F 2 "Capacitors_SMD:C_0805" H 8250 5000 50  0001 C CNN
 F 3 "" H 8250 5000 50  0001 C CNN
 	1    8250 5000
@@
 F 0 "R6" V 10330 4500 50  0000 C CNN
 F 1 "5k" V 10250 4500 50  0000 C CNN
-F 2 "Resistors_SMD:R_0402" V 10180 4500 50  0001 C CNN
+F 2 "Resistors_SMD:R_0805" V 10180 4500 50  0001 C CNN
 F 3 "" H 10250 4500 50  0001 C CNN
 	1    10250 4500
@@
 F 0 "C13" H 4110 3720 50  0000 L CNN
 F 1 "1uF" H 4110 3570 50  0000 L CNN
-F 2 "Capacitors_SMD:C_0402" H 4100 3650 50  0001 C CNN
+F 2 "Capacitors_SMD:C_0805" H 4100 3650 50  0001 C CNN
 F 3 "" H 4100 3650 50  0001 C CNN
 	1    4100 3650
@@
 F 0 "R4" V 5730 3900 50  0000 C CNN
 F 1 "10k" V 5650 3900 50  0000 C CNN
-F 2 "Resistors_SMD:R_0402" V 5580 3900 50  0001 C CNN
+F 2 "Resistors_SMD:R_0805" V 5580 3900 50  0001 C CNN
 F 3 "" H 5650 3900 50  0001 C CNN
 	1    5650 3900
@@
 F 0 "C212" H 4210 5670 50  0000 L CNN
 F 1 "0.47uF" H 4210 5520 50  0000 L CNN
-F 2 "Capacitors_SMD:C_0402" H 4200 5600 50  0001 C CNN
+F 2 "Capacitors_SMD:C_0805" H 4200 5600 50  0001 C CNN
 F 3 "" H 4200 5600 50  0001 C CNN
 	1    4200 5600
@@
 F 0 "C213" H 5710 5170 50  0000 L CNN
 F 1 "0.01uF" H 5710 5020 50  0000 L CNN
-F 2 "Capacitors_SMD:C_0201" H 5700 5100 50  0001 C CNN
+F 2 "Capacitors_SMD:C_1206" H 5700 5100 50  0001 C CNN
 F 3 "" H 5700 5100 50  0001 C CNN
 	1    5700 5100
