File: KiCad_files/RASAC.sch (KiCad schematic (older format))
At the start: 0 parts

Commit message: Purged RAM (SCH)
Was taking way too lon of a time which I didn't have
Also using larger resistors and capacitors than 0402 and 0201 (expect a very few)
Changed lines of the file:
@@
 $Descr A 11000 8500
 encoding utf-8
-Sheet 1 9
+Sheet 1 7
 Title "Reconfigurable Application-Specific Accelerator Card"
-Date "2019-02-27"
-Rev "1.0"
+Date "2019-03-31"
+Rev "0.9"
 Comp "Brian Hong & Jasmine Tang"
 Comment1 ""
@@
 $EndSheet
 $Sheet
-S 4800 4550 1550 950
-U 5C0652F6
-F0 "DDR2_1" 60
-F1 "DDR2_1.sch" 60
-$EndSheet
-$Sheet
-S 6600 4550 1550 950
-U 5C14AAFF
-F0 "DDR2_2" 60
-F1 "DDR2_2.sch" 60
-$EndSheet
-$Sheet
